File: usb-c-pd.kicad_sch (KiCad schematic)
At the start: 51 parts, among them J2 Barrel_Jack_Switch, J3 Conn_ARM_SWD_TagConnect_TC203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, J4 USB_C_Receptacle_USB2.0_14P, Q1 T2N7002AK, U1 CYPD3177-24LQ, U2 STM32C071F8Px, U3 INA180A2, U4 XL1509-3.3

Commit message: feat: preliminary layout
Parts:
- added C16: 4.7uF, Capacitor_SMD:C_0603_1608Metric_Pad1.08x0.95mm_HandSolder, symbol Device:C_Small
- D3: footprint Diode_THT:D_DO-201AD_P15.24mm_Horizontal -> Diode_SMD:D_0603_1608Metric_Pad1.05x0.95mm_HandSolder
- J1: renamed from J4; footprint (none) -> Connector_USB:USB_C_Receptacle_Amphenol_12401948E412A; symbol Connector:USB_C_Receptacle_USB2.0_14P -> Connector:USB_C_Receptacle_USB2.0_16P
- R5: value TODO -> 20k
Connections:
- net GND: now also C16.2; no longer J1.S1 (SHIELD)
- net VBUS: now also C16.1
- net VCONN: now also J2.A1
- no-connect marks 5 -> 8
Other:
- note removed: "verify this"
Changed lines of the file:
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@@
 		)
 	)
-	(text "verify this\n"
-		(exclude_from_sim no)
-		(at 52.578 154.432 0)
-		(effects
-			(font
-				(size 1.016 1.016)
-			)
-		)
-	)
 	(text "VBUX_MAX = 3V3/2 -> 15V"
 		(exclude_from_sim no)
@@
 	)
 	(junction
-		(at 33.02 168.91)
-		(diameter 0)
-		(color 0 0 0 0)
-	)
-	(junction
 		(at 194.31 24.13)
 		(diameter 0)
@@
 	)
 	(no_connect
+		(at 25.4 168.91)
+	)
+	(no_connect
+		(at 48.26 158.75)
+	)
+	(no_connect
 		(at 276.86 124.46)
 	)
 	(no_connect
+		(at 48.26 161.29)
+	)
+	(no_connect
 		(at 226.06 132.08)
 	)
@@
 	(wire
 		(pts
+			(xy 57.15 127) (xy 63.5 127)
+		)
+		(stroke
+			(width 0)
+			(type default)
+		)
+	)
+	(wire
+		(pts
 			(xy 220.98 124.46) (xy 226.06 124.46)
 		)
@@
 	(wire
 		(pts
+			(xy 68.58 127) (xy 72.39 127)
+		)
+		(stroke
+			(width 0)
+			(type default)
+		)
+	)
+	(wire
+		(pts
 			(xy 186.69 143.51) (xy 186.69 144.78)
 		)
@@
 	(wire
 		(pts
+			(xy 72.39 127) (xy 72.39 128.27)
+		)
+		(stroke
+			(width 0)
+			(type default)
+		)
+	)
+	(wire
+		(pts
 			(xy 307.34 128.27) (xy 307.34 130.81)
 		)
@@
 	(wire
 		(pts
-			(xy 25.4 168.91) (xy 33.02 168.91)
-		)
-		(stroke
-			(width 0)
-			(type default)
-		)
-	)
-	(wire
-		(pts
 			(xy 307.34 109.22) (xy 316.23 109.22)
 		)
@@
 	)
 	(symbol
+		(lib_id "power:GND")
+		(at 72.39 128.27 0)
+		(unit 1)
+		(exclude_from_sim no)
+		(in_bom yes)
+		(on_board yes)
+		(dnp no)
+		(property "Reference" "#PWR036"
+			(at 72.39 134.62 0)
+			(effects
+				(font
+					(size 1.27 1.27)
+				)
+				(hide yes)
+			)
+		)
+		(property "Value" "GND"
+			(at 72.39 132.08 0)
+			(effects
+				(font
+					(size 1.27 1.27)
+				)
+			)
+		)
+		(property "Footprint" ""
+			(at 72.39 128.27 0)
+			(effects
+				(font
+					(size 1.27 1.27)
+				)
+				(hide yes)
+			)
+		)
+		(property "Datasheet" ""
+			(at 72.39 128.27 0)
+			(effects
+				(font
+					(size 1.27 1.27)
+				)
+				(hide yes)
+			)
+		)
+		(property "Description" "Power symbol creates a global label with name \"GND\" , ground"
+			(at 72.39 128.27 0)
+			(effects
+				(font
+					(size 1.27 1.27)
+				)
+				(hide yes)
+			)
+		)
+		(pin "1"
+		)
+		(instances
+			(project "usb-c-pd"
+				(path "/8b91f438-df16-4abb-b457-7ba42e3c4b7f"
+					(reference "#PWR036")
+					(unit 1)
+				)
+			)
+		)
+	)
+	(symbol
 		(lib_id "Device:R_Small")
 		(at 62.23 71.12 0)
@@
 			)
 		)
-		(property "Value" "TODO"
+		(property "Value" "20k"
 			(at 168.91 140.97 0)
 			(effects
@@
 	)
 	(symbol
-		(lib_id "Connector:USB_C_Receptacle_USB2.0_14P")
+		(lib_id "Connector:USB_C_Receptacle_USB2.0_16P")
 		(at 33.02 146.05 0)
 		(unit 1)
@@
 		(dnp no)
 		(fields_autoplaced yes)
-		(property "Reference" "J4"
+		(property "Reference" "J1"
 			(at 33.02 123.19 0)
 			(effects
@@
 			)
 		)
-		(property "Footprint" ""
+		(property "Footprint" "Connector_USB:USB_C_Receptacle_Amphenol_12401948E412A"
 			(at 36.83 146.05 0)
 			(effects
@@
 			)
 		)
-		(property "Description" "USB 2.0-only 14P Type-C Receptacle connector"
+		(property "Description" "USB 2.0-only 16P Type-C Receptacle connector"
 			(at 33.02 146.05 0)
 			(effects
@@
 		(pin "B7"
 		)
+		(pin "A8"
+		)
+		(pin "B8"
+		)
 		(instances
 			(project ""
 				(path "/8b91f438-df16-4abb-b457-7ba42e3c4b7f"
-					(reference "J4")
+					(reference "J1")
 					(unit 1)
 				)
@@
 		(pin "3"
 		)
+		(pin "A1"
+		)
 		(instances
 			(project ""
@@
 			)
 		)
-		(property "Footprint" "Diode_THT:D_DO-201AD_P15.24mm_Horizontal"
+		(property "Footprint" "Diode_SMD:D_0603_1608Metric_Pad1.05x0.95mm_HandSolder"
 			(at 167.005 241.3 0)
 			(effects
@@
 					(unit 1)
 				)
+			)
+		)
+	)
+	(symbol
+		(lib_id "Device:C_Small")
+		(at 66.04 127 90)
+		(unit 1)
+		(exclude_from_sim no)
+		(in_bom yes)
+		(on_board yes)
+		(dnp no)
+		(property "Reference" "C16"
+			(at 63.754 120.65 90)
+			(effects
+				(font
+					(size 1.27 1.27)
+				)
+				(justify right)
+			)
+		)
+		(property "Value" "4.7uF"
+			(at 63.754 123.19 90)
+			(effects
+				(font
+					(size 1.27 1.27)
+				)
+				(justify right)
+			)
+		)
+		(property "Footprint" "Capacitor_SMD:C_0603_1608Metric_Pad1.08x0.95mm_HandSolder"
+			(at 66.04 127 0)
+			(effects
+				(font
+					(size 1.27 1.27)
+				)
+				(hide yes)
+			)
+		)
+		(property "Datasheet" "~"
+			(at 66.04 127 0)
+			(effects
+				(font
+					(size 1.27 1.27)
+				)
+				(hide yes)
+			)
+		)
+		(property "Description" "Unpolarized capacitor, small symbol"
+			(at 66.04 127 0)
+			(effects
+				(font
+					(size 1.27 1.27)
+				)
+				(hide yes)
+			)
+		)
+		(pin "2"
+		)
+		(pin "1"
+		)
+		(instances
+			(project "usb-c-pd"
+				(path "/8b91f438-df16-4abb-b457-7ba42e3c4b7f"
+					(reference "C16")
+					(unit 1)
+				)
